Commit message: Updated tentabot.urdf.xacro, realsense-d435.macro.xacro, mav_r200.gazebo: based on the namespace updates on gazebo, robot_state_publisher, gazebo_ros::spawn_model, etc.

File: urdf/realsense-d435.macro.xacro (robot description, xacro)
@@ -21,5 +21,5 @@
 <robot name="d435" xmlns:xacro="http://ros.org/wiki/xacro">
     <!--xacro:macro name="d435" params="offset_x offset_y offset_z"-->
-    <xacro:macro name="realsense-d435" params="prefix parent *origin">
+    <xacro:macro name="realsense-d435" params="prefix parent *origin ns">
         <xacro:property name="d435_cam_depth_to_left_ir_offset" value="0.0"/>
         <xacro:property name="d435_cam_depth_to_right_ir_offset" value="-0.050"/>
@@ -32,20 +32,20 @@
         <xacro:property name="d435_cam_depth_py" value="0.0175"/>
         <xacro:property name="d435_cam_depth_pz" value="${d435_cam_height/2}"/>
-        <joint name="${prefix}camera_joint" type="fixed">
+        <joint name="${prefix}/camera_joint" type="fixed">
             <parent link="${parent}"/>
-            <child link="${prefix}camera_bottom_screw_frame" />
+            <child link="${prefix}/camera_bottom_screw_frame" />
             <xacro:insert_block name="origin"/>
             <!--origin rpy="0.0 0.0 0" xyz="${offset_x} ${offset_y} ${offset_z}"/-->
         </joint>
-        <link name="${prefix}camera_bottom_screw_frame"/>
-        <gazebo reference="${prefix}camera_bottom_screw_frame">
-            <turnGravityOff>false</turnGravityOff>
-        </gazebo>
-        <joint name="${prefix}camera_link_joint" type="fixed">
+        <link name="${prefix}/camera_bottom_screw_frame"/>
+        <gazebo reference="${prefix}/camera_bottom_screw_frame">
+            <turnGravityOff>false</turnGravityOff>
+        </gazebo>
+        <joint name="${prefix}/camera_link_joint" type="fixed">
             <origin xyz="0 ${d435_cam_depth_py} ${d435_cam_depth_pz}" rpy="0 0 0"/>
-            <parent link="${prefix}camera_bottom_screw_frame"/>
-            <child link="${prefix}camera_link" />
-        </joint>
-        <link name="${prefix}camera_link">
+            <parent link="${prefix}/camera_bottom_screw_frame"/>
+            <child link="${prefix}/camera_link" />
+        </joint>
+        <link name="${prefix}/camera_link">
             <visual>
                 <origin xyz="${d435_cam_mount_from_center_offset} ${-d435_cam_depth_py} 0" rpy="${M_PI_2} 0 ${M_PI_2}"/>
@@ -68,95 +68,95 @@
         </inertial>
         </link>
-        <gazebo reference="${prefix}camera_link">
+        <gazebo reference="${prefix}/camera_link">
             <turnGravityOff>false</turnGravityOff>
             <material>Gazebo/Grey</material>
         </gazebo>
         <!-- camera depth joints and links -->
-        <joint name="${prefix}camera_depth_joint" type="fixed">
+        <joint name="${prefix}/camera_depth_joint" type="fixed">
             <origin xyz="0 0 0" rpy="0 0 0"/>
-            <parent link="${prefix}camera_link"/>
-            <child link="${prefix}camera_depth_frame" />
-        </joint>
-        <link name="${prefix}camera_depth_frame"/>
-        <gazebo reference="${prefix}camera_depth_frame">
-            <turnGravityOff>false</turnGravityOff>
-        </gazebo>
-        <joint name="${prefix}camera_depth_optical_joint" type="fixed">
-            <origin xyz="0 0 0" rpy="${-M_PI_2} 0 ${-M_PI_2}" />
-            <parent link="${prefix}camera_depth_frame" />
-            <child link="${prefix}camera_depth_optical_frame" />
-        </joint>
-        <link name="${prefix}camera_depth_optical_frame"/>
-        <gazebo reference="${prefix}camera_depth_optical_frame">
+            <parent link="${prefix}/camera_link"/>
+            <child link="${prefix}/camera_depth_frame" />
+        </joint>
+        <link name="${prefix}/camera_depth_frame"/>
+        <gazebo reference="${prefix}/camera_depth_frame">
+            <turnGravityOff>false</turnGravityOff>
+        </gazebo>
+        <joint name="${prefix}/camera_depth_optical_joint" type="fixed">
+            <origin xyz="0 0 0" rpy="${-M_PI_2} 0 ${-M_PI_2}" />
+            <parent link="${prefix}/camera_depth_frame" />
+            <child link="${prefix}/camera_depth_optical_frame" />
+        </joint>
+        <link name="${prefix}/camera_depth_optical_frame"/>
+        <gazebo reference="${prefix}/camera_depth_optical_frame">
             <turnGravityOff>false</turnGravityOff>
         </gazebo>
         <!-- camera left IR joints and links -->
-        <joint name="${prefix}camera_left_ir_joint" type="fixed">
+        <joint name="${prefix}/camera_left_ir_joint" type="fixed">
             <origin xyz="0 ${d435_cam_depth_to_left_ir_offset} 0" rpy="0 0 0" />
-            <parent link="${prefix}camera_depth_frame" />
-            <child link="${prefix}camera_left_ir_frame" />
-        </joint>
-        <link name="${prefix}camera_left_ir_frame"/>
-        <gazebo reference="${prefix}camera_left_ir_frame">
-            <turnGravityOff>false</turnGravityOff>
-        </gazebo>
-        <joint name="${prefix}camera_left_ir_optical_joint" type="fixed">
-            <origin xyz="0 0 0" rpy="${-M_PI_2} 0 ${-M_PI_2}" />
-            <parent link="${prefix}camera_left_ir_frame" />
-            <child link="${prefix}camera_left_ir_optical_frame" />
-        </joint>
-        <link name="${prefix}camera_left_ir_optical_frame"/>
-        <gazebo reference="${prefix}camera_left_ir_optical_frame">
+            <parent link="${prefix}/camera_depth_frame" />
+            <child link="${prefix}/camera_left_ir_frame" />
+        </joint>
+        <link name="${prefix}/camera_left_ir_frame"/>
+        <gazebo reference="${prefix}/camera_left_ir_frame">
+            <turnGravityOff>false</turnGravityOff>
+        </gazebo>
+        <joint name="${prefix}/camera_left_ir_optical_joint" type="fixed">
+            <origin xyz="0 0 0" rpy="${-M_PI_2} 0 ${-M_PI_2}" />
+            <parent link="${prefix}/camera_left_ir_frame" />
+            <child link="${prefix}/camera_left_ir_optical_frame" />
+        </joint>
+        <link name="${prefix}/camera_left_ir_optical_frame"/>
+        <gazebo reference="${prefix}/camera_left_ir_optical_frame">
             <turnGravityOff>false</turnGravityOff>
         </gazebo>
         <!-- camera right IR joints and links -->
-        <joint name="${prefix}camera_right_ir_joint" type="fixed">
+        <joint name="${prefix}/camera_right_ir_joint" type="fixed">
             <origin xyz="0 ${d435_cam_depth_to_right_ir_offset} 0" rpy="0 0 0" />
-            <parent link="${prefix}camera_depth_frame" />
-            <child link="${prefix}camera_right_ir_frame" />
-        </joint>
-        <link name="${prefix}camera_right_ir_frame"/>
-        <gazebo reference="${prefix}camera_right_ir_frame">
-            <turnGravityOff>false</turnGravityOff>
-        </gazebo>
-        <joint name="${prefix}camera_right_ir_optical_joint" type="fixed">
-            <origin xyz="0 0 0" rpy="${-M_PI_2} 0 ${-M_PI_2}" />
-            <parent link="${prefix}camera_right_ir_frame" />
-            <child link="${prefix}camera_right_ir_optical_frame" />
-        </joint>
-        <link name="${prefix}camera_right_ir_optical_frame"/>
-        <gazebo reference="${prefix}camera_right_ir_optical_frame">
+            <parent link="${prefix}/camera_depth_frame" />
+            <child link="${prefix}/camera_right_ir_frame" />
+        </joint>
+        <link name="${prefix}/camera_right_ir_frame"/>
+        <gazebo reference="${prefix}/camera_right_ir_frame">
+            <turnGravityOff>false</turnGravityOff>
+        </gazebo>
+        <joint name="${prefix}/camera_right_ir_optical_joint" type="fixed">
+            <origin xyz="0 0 0" rpy="${-M_PI_2} 0 ${-M_PI_2}" />
+            <parent link="${prefix}/camera_right_ir_frame" />
+            <child link="${prefix}/camera_right_ir_optical_frame" />
+        </joint>
+        <link name="${prefix}/camera_right_ir_optical_frame"/>
+        <gazebo reference="${prefix}/camera_right_ir_optical_frame">
             <turnGravityOff>false</turnGravityOff>
         </gazebo>
         <!-- camera color joints and links -->
-        <joint name="${prefix}camera_color_joint" type="fixed">
+        <joint name="${prefix}/camera_color_joint" type="fixed">
             <origin xyz="0 ${d435_cam_depth_to_color_offset} 0" rpy="0 0 0" />
-            <parent link="${prefix}camera_depth_frame" />
-            <child link="${prefix}camera_color_frame" />
-        </joint>
-        <link name="${prefix}camera_color_frame"/>
-        <gazebo reference="${prefix}camera_color_frame">
-            <turnGravityOff>false</turnGravityOff>
-        </gazebo>
-        <joint name="${prefix}camera_color_optical_joint" type="fixed">
-            <origin xyz="0 0 0" rpy="${-M_PI_2} 0 ${-M_PI_2}" />
-            <parent link="${prefix}camera_color_frame" />
-            <child link="${prefix}camera_color_optical_frame" />
-        </joint>
-        <link name="${prefix}camera_color_optical_frame"/>
-        <gazebo reference="${prefix}camera_color_optical_frame">
-            <turnGravityOff>false</turnGravityOff>
-        </gazebo>
-        <link name="${prefix}camera_depth_frame_gazebo"/>
-        <joint name="${prefix}gazebo_joint" type="fixed">
-            <origin xyz="0 0 0" rpy="${-M_PI_2} 0 ${-M_PI_2}" />
-            <parent link="${prefix}camera_link" />
-            <child link="${prefix}camera_depth_frame_gazebo" />
-        </joint>
-        <gazebo reference="camera_depth_frame_gazebo">
-            <turnGravityOff>false</turnGravityOff>
-        </gazebo>
-        <gazebo reference="${prefix}camera_link">
-        <sensor name="${prefix}d435" type="depth">
+            <parent link="${prefix}/camera_depth_frame" />
+            <child link="${prefix}/camera_color_frame" />
+        </joint>
+        <link name="${prefix}/camera_color_frame"/>
+        <gazebo reference="${prefix}/camera_color_frame">
+            <turnGravityOff>false</turnGravityOff>
+        </gazebo>
+        <joint name="${prefix}/camera_color_optical_joint" type="fixed">
+            <origin xyz="0 0 0" rpy="${-M_PI_2} 0 ${-M_PI_2}" />
+            <parent link="${prefix}/camera_color_frame" />
+            <child link="${prefix}/camera_color_optical_frame" />
+        </joint>
+        <link name="${prefix}/camera_color_optical_frame"/>
+        <gazebo reference="${prefix}/camera_color_optical_frame">
+            <turnGravityOff>false</turnGravityOff>
+        </gazebo>
+        <link name="${prefix}/camera_depth_frame_gazebo"/>
+        <joint name="${prefix}/gazebo_joint" type="fixed">
+            <origin xyz="0 0 0" rpy="${-M_PI_2} 0 ${-M_PI_2}" />
+            <parent link="${prefix}/camera_link" />
+            <child link="${prefix}/camera_depth_frame_gazebo" />
+        </joint>
+        <gazebo reference="${prefix}/camera_depth_frame_gazebo">
+            <turnGravityOff>false</turnGravityOff>
+        </gazebo>
+        <gazebo reference="${prefix}/camera_link">
+        <sensor name="${prefix}/d435" type="depth">
             <update_rate>30</update_rate>
             <camera>
@@ -178,11 +178,11 @@
                 <alwaysOn>true</alwaysOn>
                 <updateRate>0.0</updateRate>
-                <cameraName>${prefix}d435</cameraName>
-                <imageTopicName>/${prefix}d435/camera/color/image_raw</imageTopicName>
-                <cameraInfoTopicName>/${prefix}d435/camera/color/camera_info</cameraInfoTopicName>
-                <depthImageTopicName>/${prefix}d435/camera/depth/image_raw</depthImageTopicName>
-                <depthImageInfoTopicName>/${prefix}d435/camera/depth/camera_info</depthImageInfoTopicName>
-                <pointCloudTopicName>/${prefix}d435/camera/depth/color/points</pointCloudTopicName>
-                <frameName>${prefix}camera_depth_frame_gazebo</frameName>
+                <cameraName>/${ns}/${prefix}</cameraName>
+                <imageTopicName>/${ns}/${prefix}/camera/color/image_raw</imageTopicName>
+                <cameraInfoTopicName>/${ns}/${prefix}/camera/color/camera_info</cameraInfoTopicName>
+                <depthImageTopicName>/${ns}/${prefix}/camera/depth/image_raw</depthImageTopicName>
+                <depthImageInfoTopicName>/${ns}/${prefix}/camera/depth/camera_info</depthImageInfoTopicName>
+                <pointCloudTopicName>/${ns}/${prefix}/camera/depth/color/points</pointCloudTopicName>
+                <frameName>/${ns}/${prefix}/camera_depth_frame_gazebo</frameName>
                 <pointCloudCutoff>0.02</pointCloudCutoff>
                 <distortionK1>0</distortionK1>

File: urdf/tentabot.urdf.xacro (robot description, xacro)
@@ -1,6 +1,6 @@
 <?xml version="1.0" ?>
 <robot name="tentabot" xmlns:xacro="http://www.ros.org/wiki/xacro">
-    <xacro:arg name="ns" default="tentabot"/>
-    <xacro:arg name="model" default="burger"/>
+    <xacro:arg name="ns" default=""/>
+    <xacro:arg name="model" default=""/>
     <!--xacro:property name="ns" value="$(arg ns)"/-->
     <!--xacro:property name="arm_prefix" value="ur_arm_" /-->
@@ -12,8 +12,9 @@
     <!-- Import mobile base -->
     <xacro:include filename="$(find turtlebot3_description)/urdf/turtlebot3_$(arg model)_with_ns.urdf.xacro"/>
+    <!--xacro:include filename="$(find turtlebot3_description)/urdf/turtlebot3_$(arg model).urdf.xacro"/-->
     <!--xacro:include filename="$(find husky_description)/urdf/husky.urdf.xacro"/-->
     <!--xacro:include filename="$(find jackal_description)/urdf/jackal_with_ns.urdf.xacro"/-->
     <!-- Import macro for lidar-->
-    <xacro:include filename="$(find jackal_description)/urdf/accessories/sick_lms1xx_mount.urdf.xacro" />
+    <xacro:include filename="$(find lms1xx)/urdf/sick_lms1xx_mount.urdf.xacro" />
     <!-- Create lidar instance (jackal)-->
     <!--xacro:sick_lms1xx_mount prefix="$(arg ns)/front"
@@ -33,10 +34,11 @@
     <!-- Create camera instance 1.570796327 (turtlebot3 burger)-->
     <xacro:realsense-d435
-        prefix="$(arg ns)/d435_cam1"
-        parent="$(arg ns)/base_link">
+        ns="$(arg ns)"
+        prefix="d435_cam1"
+        parent="base_link">
         <origin xyz="-0.05 0.0 0.18" rpy="0.0 0.0 0.0" />
     </xacro:realsense-d435>
     <!-- Create macro for collision objects-->
-    <xacro:macro name="bumper" params="link_name radius length x y">
+    <!--xacro:macro name="bumper" params="link_name radius length x y">
         <link name="${link_name}">
             <inertial>
@@ -66,5 +68,5 @@
             <child link="${link_name}"/>
         </joint>
-    </xacro:macro>
+    </xacro:macro-->
     <!-- Create contact object -->
     <!--xacro:bumper
@@ -241,5 +243,5 @@
                 <box size="0.01 0.01 0.01"/>
             </geometry>
-        </visual>
+        </visual>${prefix}
 	</link>
     <gazebo reference="theta_link">
