Commit message: Implementation and data of IROS22 submission.

File: models/jackals/jackal_cam_depth.urdf.xacro (robot description, xacro)
@@ -222,14 +222,14 @@
   </joint>
   <!-- Bring in simulation data for Gazebo. -->
-  <xacro:include filename="$(find hybrid_rl_training)/models/jackals/jackal.gazebo" />
+  <xacro:include filename="$(find tentabot)/models/jackals/jackal.gazebo" />
   <!-- Optional standard accessories, including their simulation data. The rendering
        of these into the final description is controlled by optenv variables, which
        default each one to off.-->
   <xacro:include filename="$(find jackal_description)/urdf/accessories.urdf.xacro" />
-  <xacro:include filename="$(find hybrid_rl_training)/models/realsense2_description/urdf/d435_depth.macro.xacro" />
+  <xacro:include filename="$(find tentabot)/models/realsense2_description/urdf/d435_depth.macro.xacro" />
   <xacro:sensor_d435 prefix="" parent="rear_mount">
     <origin xyz="0 0 1" rpy="0 0 0"/>
   </xacro:sensor_d435>
-  <xacro:include filename="$(find hybrid_rl_training)/models/hokuyo/hokuyo.urdf.xacro"/>
+  <xacro:include filename="$(find tentabot)/models/hokuyo/hokuyo.urdf.xacro"/>
   <xacro:sensor_hokuyo prefix="" parent="front_mount">
     <origin xyz="0 0 0.02" rpy="0 0 0"/>

File: models/jackals/jackal_cam_mono.urdf.xacro (robot description, xacro)
@@ -222,10 +222,10 @@
   </joint>
   <!-- Bring in simulation data for Gazebo. -->
-  <xacro:include filename="$(find navisim)/models/jackals/jackal.gazebo" />
+  <xacro:include filename="$(find tentabot)/models/jackals/jackal.gazebo" />
   <!-- Optional standard accessories, including their simulation data. The rendering
        of these into the final description is controlled by optenv variables, which
        default each one to off.-->
   <xacro:include filename="$(find jackal_description)/urdf/accessories.urdf.xacro" />
-  <xacro:include filename="$(find navisim)/models/realsense2_description/urdf/d435_mono.macro.xacro" />
+  <xacro:include filename="$(find tentabot)/models/realsense2_description/urdf/d435_mono.macro.xacro" />
   <xacro:sensor_d435 prefix="/$(arg namespace)" parent="rear_mount">
     <origin xyz="0 0 1" rpy="0 0 0"/>

File: models/jackals/jackal_multi.urdf.xacro (robot description, xacro)
@@ -222,5 +222,5 @@
   </joint>
   <!-- Bring in simulation data for Gazebo. -->
-  <xacro:include filename="$(find navisim)/models/jackals/jackal.gazebo" />
+  <xacro:include filename="$(find tentabot)/models/jackals/jackal.gazebo" />
   <!-- Optional standard accessories, including their simulation data. The rendering
        of these into the final description is controlled by optenv variables, which

File: models/jackals/jackal_single.urdf.xacro (robot description, xacro)
@@ -227,7 +227,7 @@
        default each one to off.-->
   <xacro:include filename="$(find jackal_description)/urdf/accessories.urdf.xacro" />
-  <xacro:include filename="$(find navisim)/models/realsense2_description/urdf/_d435.macro.xacro" />
+  <xacro:include filename="$(find tentabot)/models/realsense2_description/urdf/_d435.macro.xacro" />
   <xacro:sensor_d435 prefix="" parent="rear_mount">
-    <origin xyz="0 0 1" rpy="0 0 0"/>
+    <origin xyz="0 0 0" rpy="0 0 0"/>
   </xacro:sensor_d435>
 </robot>

File: models/turtlebot2/kobuki/kobuki.urdf.xacro (robot description, xacro)
@@ -7,6 +7,6 @@
  -->
 <robot name="kobuki" xmlns:xacro="http://ros.org/wiki/xacro">
-  <xacro:include filename="$(find tentabot_devel)/models/turtlebot2/common_properties.urdf.xacro"/>
-  <xacro:include filename="$(find tentabot_devel)/models/turtlebot2/kobuki/kobuki_gazebo.urdf.xacro"/>
+  <xacro:include filename="$(find tentabot)/models/turtlebot2/common_properties.urdf.xacro"/>
+  <xacro:include filename="$(find tentabot)/models/turtlebot2/kobuki/kobuki_gazebo.urdf.xacro"/>
   <!-- Kobuki -->
   <xacro:macro name="kobuki">

File: models/turtlebot2/sensors/hokuyo.urdf.xacro (robot description, xacro)
@@ -12,5 +12,5 @@
         <origin xyz="0 0 0" rpy="0 0 0"/>
         <geometry>
-          <mesh filename="package://tentabot_devel/models/hokuyo/hokuyo.dae"/>
+          <mesh filename="package://tentabot/models/hokuyo/hokuyo.dae"/>
         </geometry>
       </visual>

File: models/turtlebot2/sensors/r200.urdf.xacro (robot description, xacro)
@@ -2,5 +2,5 @@
 <robot name="sensor_r200" xmlns:xacro="http://ros.org/wiki/xacro">
   <!--xacro:include filename="$(find navisim)/models/turtlebot2/turtlebot_gazebo.urdf.xacro"/-->
-  <xacro:include filename="$(find tentabot_devel)/models/turtlebot2/common_properties.urdf.xacro"/>
+  <xacro:include filename="$(find tentabot)/models/turtlebot2/common_properties.urdf.xacro"/>
   <!-- Mount and camera parameters -->
   <xacro:property name="pole_px" value="-0.103" />

File: models/turtlebot2/turtlebot.urdf.xacro (robot description, xacro)
@@ -6,13 +6,13 @@
 -->
 <robot name="turtlebot" xmlns:xacro="http://ros.org/wiki/xacro">
-  <xacro:include filename="$(find tentabot_devel)/models/turtlebot2/common_properties.urdf.xacro" />
-  <xacro:include filename="$(find tentabot_devel)/models/turtlebot2/kobuki/kobuki.urdf.xacro" />
-  <xacro:include filename="$(find tentabot_devel)/models/turtlebot2/stacks/hexagons.urdf.xacro"/>
+  <xacro:include filename="$(find tentabot)/models/turtlebot2/common_properties.urdf.xacro" />
+  <xacro:include filename="$(find tentabot)/models/turtlebot2/kobuki/kobuki.urdf.xacro" />
+  <xacro:include filename="$(find tentabot)/models/turtlebot2/stacks/hexagons.urdf.xacro"/>
   <!--sensors-->
-  <xacro:include filename="$(find tentabot_devel)/models/turtlebot2/sensors/hokuyo.urdf.xacro"/>
-  <xacro:include filename="$(find tentabot_devel)/models/turtlebot2/sensors/r200.urdf.xacro"/>
+  <xacro:include filename="$(find tentabot)/models/turtlebot2/sensors/hokuyo.urdf.xacro"/>
+  <xacro:include filename="$(find tentabot)/models/turtlebot2/sensors/r200.urdf.xacro"/>
   <!--xacro:include filename="$(find slam_ros)/models/urdf/sensors/asus_xtion_pro.urdf.xacro"/>
   <xacro:include filename="$(find slam_ros)/models/urdf/sensors/asus_xtion_pro_offset.urdf.xacro"/-->
-  <kobuki/>
+  <xacro:kobuki/>
   <stack_hexagons parent="base_link"/>
   <sensor_r200  parent="base_link"/>

File: urdf/materials.xacro (robot description, xacro)
@@ -50,6 +50,6 @@
         <color rgba="0.9 0.9 0.9 1.0" />
     </material>
-    <material name="dark_grey">
+    <!--material name="dark_grey">
       <color rgba="0.3 0.3 0.3 1"/>
-    </material>
+    </material-->
 </robot>

File: urdf/realsense-d435.macro.xacro (robot description, xacro)
@@ -20,6 +20,5 @@
 -->
 <robot name="d435" xmlns:xacro="http://ros.org/wiki/xacro">
-    <!--xacro:macro name="d435" params="offset_x offset_y offset_z"-->
-    <xacro:macro name="realsense-d435" params="prefix parent *origin ns">
+    <xacro:macro name="realsense-d435" params="prefix parent *origin">
         <xacro:property name="d435_cam_depth_to_left_ir_offset" value="0.0"/>
         <xacro:property name="d435_cam_depth_to_right_ir_offset" value="-0.050"/>
@@ -36,5 +35,4 @@
             <child link="${prefix}/camera_bottom_screw_frame" />
             <xacro:insert_block name="origin"/>
-            <!--origin rpy="0.0 0.0 0" xyz="${offset_x} ${offset_y} ${offset_z}"/-->
         </joint>
         <link name="${prefix}/camera_bottom_screw_frame"/>
@@ -178,11 +176,11 @@
                 <alwaysOn>true</alwaysOn>
                 <updateRate>0.0</updateRate>
-                <cameraName>/${ns}/${prefix}</cameraName>
-                <imageTopicName>/${ns}/${prefix}/camera/color/image_raw</imageTopicName>
-                <cameraInfoTopicName>/${ns}/${prefix}/camera/color/camera_info</cameraInfoTopicName>
-                <depthImageTopicName>/${ns}/${prefix}/camera/depth/image_raw</depthImageTopicName>
-                <depthImageInfoTopicName>/${ns}/${prefix}/camera/depth/camera_info</depthImageInfoTopicName>
-                <pointCloudTopicName>/${ns}/${prefix}/camera/depth/color/points</pointCloudTopicName>
-                <frameName>/${ns}/${prefix}/camera_depth_frame_gazebo</frameName>
+                <cameraName>${prefix}</cameraName>
+                <imageTopicName>${prefix}/camera/color/image_raw</imageTopicName>
+                <cameraInfoTopicName>${prefix}/camera/color/camera_info</cameraInfoTopicName>
+                <depthImageTopicName>${prefix}/camera/depth/image_raw</depthImageTopicName>
+                <depthImageInfoTopicName>${prefix}/camera/depth/camera_info</depthImageInfoTopicName>
+                <pointCloudTopicName>${prefix}/camera/depth/color/points</pointCloudTopicName>
+                <frameName>${prefix}/camera_depth_frame_gazebo</frameName>
                 <pointCloudCutoff>0.02</pointCloudCutoff>
                 <distortionK1>0</distortionK1>
